File: Macropad.kicad_pcb (KiCad board)
At the start: 2 copper layers, 84.8 x 63.2 mm, 19 parts, among them U1 Arduino_Pro_Micro

Commit message: Update PCB
Parts:
- added SW1: Switch, Button_Switch_THT:SW_PUSH_6mm, F.Cu at (116.5, 102.8)
Connections:
- U1 pad 22: unconnected-(U1-RST-Pad22) -> Net-(U1-RST)
- U1 pad 23: unconnected-(U1-GND-Pad23) -> GND
- U1 pad 3: unconnected-(U1-GND-Pad3) -> GND
- U1 pad 4: unconnected-(U1-GND-Pad4) -> GND
Routing:
- net Net-(U1-RST): track 0.00 -> 36.7 mm
- added copper zone on F.Cu, net GND
- removed copper zone on B.Cu, net (none)
- removed copper zone on F.Cu, net (none)
